File: pcb/CPU.kicad_sch (KiCad schematic)
At the start: 32 parts, among them J2 USB_C_Receptacle_USB2.0_16P, U1 F1C100s, Y1 24MHz

Commit message: Added bom and fixed PCB with LCSC numbers
Parts:
- C1, C10, C11, C16: LCSC# (none) -> C12530
- C12, C13, C14, C15, C17, C18, C2, C21, C3, C4, C5, C6, C7, C8, C9: LCSC# (none) -> C1525
- C19, C20: value C -> 12p; LCSC# (none) -> C26406
- R3, R4: LCSC# (none) -> C105872
- R5: LCSC# (none) -> C93943
- R6, R7: LCSC# (none) -> C114765
- R8, R9: LCSC# (none) -> C60488
- Y1: LCSC# (none) -> C7303340
Changed lines of the file:
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@@
 			)
 		)
-		(property "LCSC#" ""
+		(property "LCSC#" "C105872"
 			(at 256.54 35.56 90)
 			(hide yes)
@@
 			)
 		)
-		(property "LCSC#" ""
+		(property "LCSC#" "C1525"
 			(at 146.05 33.02 0)
 			(hide yes)
@@
 			)
 		)
-		(property "LCSC#" ""
+		(property "LCSC#" "C1525"
 			(at 69.85 33.02 0)
 			(hide yes)
@@
 			)
 		)
-		(property "LCSC#" ""
+		(property "LCSC#" "C114765"
 			(at 161.29 82.55 90)
 			(hide yes)
@@
 			)
 		)
-		(property "LCSC#" ""
+		(property "LCSC#" "C105872"
 			(at 256.54 38.1 90)
 			(hide yes)
@@
 			)
 		)
-		(property "LCSC#" ""
+		(property "LCSC#" "C93943"
 			(at 34.29 53.34 0)
 			(hide yes)
@@
 			)
 		)
+		(property "LCSC#" "C60488"
+			(at 201.93 102.87 0)
+			(hide yes)
+			(show_name no)
+			(do_not_autoplace no)
+			(effects
+				(font
+					(size 1.27 1.27)
+				)
+			)
+		)
 		(pin "2"
 		)
@@
 			)
 		)
-		(property "LCSC#" ""
+		(property "LCSC#" "C1525"
 			(at 104.14 57.15 0)
 			(hide yes)
@@
 			)
 		)
+		(property "LCSC#" "C60488"
+			(at 201.93 113.03 0)
+			(hide yes)
+			(show_name no)
+			(do_not_autoplace no)
+			(effects
+				(font
+					(size 1.27 1.27)
+				)
+			)
+		)
 		(pin "2"
 		)
@@
 			)
 		)
-		(property "LCSC#" ""
+		(property "LCSC#" "C1525"
 			(at 143.51 57.15 0)
 			(hide yes)
@@
 			)
 		)
-		(property "Value" "C"
+		(property "Value" "12p"
 			(at 52.07 106.6799 0)
 			(show_name no)
@@
 			)
 		)
-		(property "LCSC#" ""
+		(property "LCSC#" "C26406"
 			(at 48.26 105.41 0)
 			(hide yes)
@@
 			)
 		)
-		(property "Value" "C"
+		(property "Value" "12p"
 			(at 31.75 106.6799 0)
 			(show_name no)
@@
 			)
 		)
-		(property "LCSC#" ""
+		(property "LCSC#" "C26406"
 			(at 35.56 105.41 0)
 			(hide yes)
@@
 			)
 		)
-		(property "LCSC#" ""
+		(property "LCSC#" "C1525"
 			(at 125.73 33.02 0)
 			(hide yes)
@@
 			)
 		)
-		(property "LCSC#" ""
+		(property "LCSC#" "C7303340"
 			(at 41.91 99.06 0)
 			(hide yes)
@@
 			)
 		)
-		(property "LCSC#" ""
+		(property "LCSC#" "C1525"
 			(at 133.35 57.15 0)
 			(hide yes)
@@
 			)
 		)
-		(property "LCSC#" ""
+		(property "LCSC#" "C12530"
 			(at 156.21 33.02 0)
 			(hide yes)
@@
 			)
 		)
-		(property "LCSC#" ""
+		(property "LCSC#" "C12530"
 			(at 59.69 33.02 0)
 			(hide yes)
@@
 			)
 		)
-		(property "LCSC#" ""
+		(property "LCSC#" "C12530"
 			(at 163.83 57.15 0)
 			(hide yes)
@@
 			)
 		)
-		(property "LCSC#" ""
+		(property "LCSC#" "C1525"
 			(at 153.67 57.15 0)
 			(hide yes)
@@
 			)
 		)
+		(property "LCSC#" "C1525"
+			(at 212.09 102.87 0)
+			(hide yes)
+			(show_name no)
+			(do_not_autoplace no)
+			(effects
+				(font
+					(size 1.27 1.27)
+				)
+			)
+		)
 		(pin "1"
 		)
@@
 			)
 		)
-		(property "LCSC#" ""
+		(property "LCSC#" "C1525"
 			(at 100.33 33.02 0)
 			(hide yes)
@@
 			)
 		)
-		(property "LCSC#" ""
+		(property "LCSC#" "C1525"
 			(at 80.01 33.02 0)
 			(hide yes)
@@
 			)
 		)
-		(property "LCSC#" ""
+		(property "LCSC#" "C1525"
 			(at 90.17 33.02 0)
 			(hide yes)
@@
 			)
 		)
-		(property "LCSC#" ""
+		(property "LCSC#" "C1525"
 			(at 135.89 33.02 0)
 			(hide yes)
@@
 			)
 		)
-		(property "LCSC#" ""
+		(property "LCSC#" "C1525"
 			(at 110.49 33.02 0)
 			(hide yes)
@@
 			)
 		)
-		(property "LCSC#" ""
+		(property "LCSC#" "C12530"
 			(at 93.98 57.15 0)
 			(hide yes)
@@
 			)
 		)
-		(property "LCSC#" ""
+		(property "LCSC#" "C114765"
 			(at 161.29 80.01 90)
 			(hide yes)
@@
 			)
 		)
+		(property "LCSC#" "C1525"
+			(at 212.09 113.03 0)
+			(hide yes)
+			(show_name no)
+			(do_not_autoplace no)
+			(effects
+				(font
+					(size 1.27 1.27)
+				)
+			)
+		)
 		(pin "1"
 		)
@@
 			)
 		)
-		(property "LCSC#" ""
+		(property "LCSC#" "C1525"
 			(at 34.29 63.5 0)
 			(hide yes)
