File: pcb/MICROCONTROLLER.kicad_sch (KiCad schematic)
At the start: 14 parts, among them J4 USB_C_Receptacle_USB2.0_16P, U3 CH343P, U4 ATmega328P-MM, Y2 24MHz

Commit message: Completed PCB
Parts:
- removed R19, R20: 22R, Resistor_SMD:R_0402_1005Metric, symbol Device:R
- added C36, C37: 100n, Capacitor_SMD:C_0402_1005Metric, symbol Device:C
- C35: footprint (none) -> Capacitor_SMD:C_0402_1005Metric
Connections:
- net USB-D+ is gone; now on net D+: J4.A6 (D+), J4.B6 (D+)
- net USB-D- is gone; now on net D-: J4.A7 (D-), J4.B7 (D-)
- net +3V3: now also U4.17 (AREF), C36.1, C37.1
- net GND: now also C35.1, C36.2, C37.2; no longer C35.2
- net XTAL1: now also Y2.1; no longer Y2.3
- net XTAL2: now also Y2.3; no longer Y2.1
- net at U3.6 (V3_{OUT}): now also C35.2; no longer C35.1
- no-connect marks 9 -> 22

Commit message: Added bom and fixed PCB with LCSC numbers
Parts:
- C31, C32: value C -> 12p; LCSC# (none) -> C26406
- C33, C34, C35, C36, C37: LCSC# (none) -> C1525
- J4: LCSC# C165948 -> C7450621
- R17, R18: LCSC# (none) -> C105872
- U3: LCSC# (none) -> C2846043
- U4: LCSC# (none) -> C2651959
- Y2: LCSC# (none) -> C7303340
Changed lines of the file:
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@@
+			)
+		)
+		(property "LCSC#" "C2651959"
+			(at 91.44 110.49 0)
+			(hide yes)
+			(show_name no)
+			(do_not_autoplace no)
+			(effects
+				(font
+					(size 1.27 1.27)
+				)
 			)
 		)
@@
 			)
 		)
-		(property "Value" "C"
+		(property "Value" "12p"
 			(at 49.53 116.8399 0)
 			(show_name no)
@@
 			)
 		)
-		(property "LCSC#" ""
+		(property "LCSC#" "C26406"
 			(at 53.34 115.57 0)
 			(hide yes)
@@
 			)
 		)
+		(property "LCSC#" "C2846043"
+			(at 142.24 69.85 0)
+			(hide yes)
+			(show_name no)
+			(do_not_autoplace no)
+			(effects
+				(font
+					(size 1.27 1.27)
+				)
+			)
+		)
 		(pin "12"
 		)
@@
 			)
 		)
-		(property "Value" "C"
+		(property "Value" "12p"
 			(at 69.85 116.8399 0)
 			(show_name no)
@@
 			)
 		)
-		(property "LCSC#" ""
+		(property "LCSC#" "C26406"
 			(at 66.04 115.57 0)
 			(hide yes)
@@
 			)
 		)
-		(property "LCSC#" ""
+		(property "LCSC#" "C1525"
 			(at 149.86 27.94 0)
 			(hide yes)
@@
 			)
 		)
-		(property "LCSC#" ""
+		(property "LCSC#" "C7303340"
 			(at 59.69 109.22 0)
 			(hide yes)
@@
 			)
 		)
-		(property "LCSC#" "C165948"
+		(property "LCSC#" "C7450621"
 			(at 233.68 52.07 0)
 			(hide yes)
@@
 			)
 		)
-		(property "LCSC#" ""
+		(property "LCSC#" "C105872"
 			(at 255.27 44.45 90)
 			(hide yes)
@@
 			)
 		)
-		(property "LCSC#" ""
+		(property "LCSC#" "C1525"
 			(at 135.89 44.45 0)
 			(hide yes)
@@
 			)
 		)
-		(property "LCSC#" ""
+		(property "LCSC#" "C1525"
 			(at 88.9 60.96 0)
 			(hide yes)
@@
 			)
 		)
-		(property "LCSC#" ""
+		(property "LCSC#" "C1525"
 			(at 77.47 60.96 0)
 			(hide yes)
@@
 			)
 		)
-		(property "LCSC#" ""
+		(property "LCSC#" "C105872"
 			(at 255.27 41.91 90)
 			(hide yes)
@@
 			)
 		)
-		(property "LCSC#" ""
+		(property "LCSC#" "C1525"
 			(at 148.59 44.45 0)
 			(hide yes)
