File: pcb/PMIC.kicad_sch (KiCad schematic)
At the start: 19 parts, among them U2 TMI7003C

Commit message: Added bom and fixed PCB with LCSC numbers
Parts:
- C22, C25, C28: LCSC# (none) -> C368809
- C23, C26, C29: LCSC# (none) -> C70464
- C24, C27, C30: LCSC# (none) -> C19702
- R10, R12, R14: LCSC# (none) -> C107229
- R11: LCSC# (none) -> C93940
- R13: LCSC# (none) -> C114761
- R15: LCSC# (none) -> C137950
Changed lines of the file:
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@@
 			)
 		)
-		(property "LCSC#" ""
+		(property "LCSC#" "C70464"
 			(at 189.23 68.58 0)
 			(hide yes)
@@
 			)
 		)
-		(property "LCSC#" ""
+		(property "LCSC#" "C107229"
 			(at 198.12 95.25 0)
 			(hide yes)
@@
 			)
 		)
-		(property "LCSC#" ""
+		(property "LCSC#" "C19702"
 			(at 208.28 68.58 0)
 			(hide yes)
@@
 			)
 		)
-		(property "LCSC#" ""
+		(property "LCSC#" "C93940"
 			(at 198.12 78.74 0)
 			(hide yes)
@@
 			)
 		)
-		(property "LCSC#" ""
+		(property "LCSC#" "C107229"
 			(at 198.12 121.92 0)
 			(hide yes)
@@
 			)
 		)
-		(property "LCSC#" ""
+		(property "LCSC#" "C368809"
 			(at 140.97 85.09 0)
 			(hide yes)
@@
 			)
 		)
-		(property "LCSC#" ""
+		(property "LCSC#" "C114761"
 			(at 198.12 105.41 0)
 			(hide yes)
@@
 			)
 		)
-		(property "LCSC#" ""
+		(property "LCSC#" "C70464"
 			(at 189.23 121.92 0)
 			(hide yes)
@@
 			)
 		)
-		(property "LCSC#" ""
+		(property "LCSC#" "C19702"
 			(at 208.28 121.92 0)
 			(hide yes)
@@
 			)
 		)
-		(property "LCSC#" ""
+		(property "LCSC#" "C137950"
 			(at 198.12 132.08 0)
 			(hide yes)
@@
 			)
 		)
-		(property "LCSC#" ""
+		(property "LCSC#" "C70464"
 			(at 189.23 95.25 0)
 			(hide yes)
@@
 			)
 		)
-		(property "LCSC#" ""
+		(property "LCSC#" "C368809"
 			(at 140.97 68.58 0)
 			(hide yes)
@@
 			)
 		)
-		(property "LCSC#" ""
+		(property "LCSC#" "C368809"
 			(at 140.97 101.6 0)
 			(hide yes)
@@
 			)
 		)
-		(property "LCSC#" ""
+		(property "LCSC#" "C19702"
 			(at 208.28 95.25 0)
 			(hide yes)
@@
 			)
 		)
-		(property "LCSC#" ""
+		(property "LCSC#" "C107229"
 			(at 198.12 68.58 0)
 			(hide yes)
