File: pcb/SD_CARD.kicad_sch (KiCad schematic)
At the start: 3 parts, among them J3 Micro_SD_Card

Commit message: Added bom and fixed PCB with LCSC numbers
Parts:
- R16: LCSC# (none) -> C93943
Changed lines of the file:
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@@
 			)
 		)
-		(property "LCSC#" ""
+		(property "LCSC#" "C93943"
 			(at 85.09 86.36 0)
 			(hide yes)
