File: pcb/linux_soc.kicad_sch (KiCad schematic)
At the start: 3 parts

Commit message: Completed PCB
Parts:
- added R19, R20: 4k7, Resistor_SMD:R_0402_1005Metric, symbol Device:R
Connections:
- net +3V3: now also R19.1, R20.1
- net I2C_SCL: now also R19.2
- net I2C_SDA: now also R20.2

Commit message: Added bom and fixed PCB with LCSC numbers
Parts:
- R1, R2: LCSC# (none) -> C106235
- R19, R20: LCSC# (none) -> C105871
Changed lines of the file:
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@@
 			)
 		)
-		(property "LCSC#" ""
+		(property "LCSC#" "C105871"
 			(at 58.42 71.12 0)
 			(hide yes)
@@
 			)
 		)
-		(property "LCSC#" ""
+		(property "LCSC#" "C106235"
 			(at 20.32 72.39 0)
 			(hide yes)
@@
 			)
 		)
-		(property "LCSC#" ""
+		(property "LCSC#" "C106235"
 			(at 27.94 72.39 0)
 			(hide yes)
@@
 			)
 		)
-		(property "LCSC#" ""
+		(property "LCSC#" "C105871"
 			(at 66.04 71.12 0)
 			(hide yes)
